File: hardware/pcb/kicad/controller.kicad_pcb (KiCad board)
At the start: 8 copper layers, 160 x 130 mm, 114 parts, among them J1 48V INPUT, J10 DUAL ESTOP LOOP, J11 SAFETY OUTPUT, J12 DUAL MANUAL RESET, J13 WCH DEBUG, J2 12V MOTOR AUX, J3 JETSON DEVKIT 12V, J4 JETSON MCU BACKPLANE, J5 CAN A, J6 CAN B, K1 FORCE-GUIDED 12V A, K2 FORCE-GUIDED 12V B, Q1 150V N-MOS, Q2 150V N-MOS, U1 LTC4368HMS-2, U2 ISOLATED 48V-12V 240W (TBD), U3 TPS26633RGE, U4 RPL-5.0 3V3/5A, U5 CH32V307VCT6, U6 ISO1042DW, U7 3V3-5V ISO 1W, U8 ESTOP DIAGNOSTIC OPTO, Y1 8MHz

Commit message: feat(hardware): implement EVT1 PCB power candidates
Parts:
- added TP10: 3V3_PGOOD, TestPoint_Pad_D1.5mm, F.Cu at (101.0, 62.0)
- added TP11: JETSON_PGOOD, TestPoint_Pad_D1.5mm, F.Cu at (102.0, 3.00)
- added TP12: JETSON_FAULT_N, TestPoint_Pad_D1.5mm, F.Cu at (108.0, 3.00)
- added TP13: U3_IMON, TestPoint_Pad_D1.5mm, F.Cu at (121.0, 3.00)
- added TP14: ESTOP_A_MON, TestPoint_Pad_D1.5mm, F.Cu at (48.0, 82.0)
- added TP15: ESTOP_B_MON, TestPoint_Pad_D1.5mm, F.Cu at (54.0, 82.0)
- added TP9: 5V_CAN_ISO, TestPoint_Pad_D1.5mm, F.Cu at (151.0, 12.0)
- C2, C6, R47, R51, RPG3, RS1, RSH1: moved to B.Cu
- U2: value ISOLATED 48V-12V 240W (TBD) -> 18-75V TO 12V 240W ISO; footprint Isolated_48V_12V_240W_TBD -> Delta_Q36SR_QuarterBrick
- U7: footprint Converter_DCDC_muRata_MEJ1SxxxxSC_THT -> Murata_NXF1_MC
- moved J3 26.5 mm to (117.5, 32.5)
- moved RS1 22.0 mm to (39.5, 43.0)
- moved C2 19.5 mm to (42.0, 51.0)
- moved C3 17.0 mm to (105.0, 39.0)
- moved C43 4.00 mm to (144.7, 14.0)
- moved C42 3.58 mm to (132.5, 14.5), turned to 180 degrees
- moved U7 3.50 mm to (135.5, 24.0)
- moved U2 2.24 mm to (68.0, 26.0)
Connections:
- U2 pad 3: (no net) -> GND_PWR
- U2 pad 4: 12V_ISO -> GND
- U2 pad 7: (no net) -> 12V_ISO
- U2 pad 8: (no net) -> 12V_ISO
- U7 pad 1: 3V3_LOGIC -> GND
- U7 pad 7: 5V_CAN_ISO -> GND_CAN_ISO
Routing:
- net 3V3_LOGIC: track 487.8 -> 395.8 mm, vias 9 -> 13
- net VBAT_PROTECTED: track 100.1 -> 176.8 mm, vias 5 -> 12
- net GND_PWR: track 122.9 -> 169.7 mm, vias 1 -> 10
- net INPUT_SENSE: track 21.7 -> 64.5 mm, vias 2 -> 4
- net GND: track 582.5 -> 611.9 mm, vias 38 -> 40
- net JETSON_PGOOD: track 29.4 -> 53.3 mm, vias 2 -> 4
- net 3V3_PGOOD: track 1.25 -> 25.1 mm, vias 0 -> 2
- net 5V_CAN_ISO: track 50.6 -> 73.2 mm, vias 1 -> 2
- net ESTOP_A_MON: track 78.0 -> 96.7 mm, vias 3 -> 5
- net JETSON_FAULT_N: track 36.9 -> 54.7 mm, vias 2 -> 4
- net ESTOP_B_MON: track 72.2 -> 88.9 mm, vias 3 -> 5
- net 12V_ISO: track 211.8 -> 226.2 mm, vias 10 -> 12
- net JETSON_12V: track 141.9 -> 127.9 mm
- net U3_IMON: track 8.67 -> 19.2 mm, vias 0 -> 2
- net GND_CAN_ISO: track 73.2 -> 83.4 mm, vias 5 -> 6
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Other:
- board text added: "U2 Q36SR 12V / 20A"
- board text added: "VERIFY EXACT DATASHEET + AVL"
- board text removed: "DO NOT FIT"
- board text removed: "U2 LAND PATTERN TBD"
