File: hardware/pcb/kicad/controller.kicad_sch (KiCad schematic)
At the start: 110 parts, among them J1 48V INPUT, J10 DUAL ESTOP LOOP, J11 SAFETY OUTPUT, J12 DUAL MANUAL RESET, J13 WCH DEBUG, J2 12V MOTOR AUX, J3 JETSON DEVKIT 12V, J4 JETSON MCU BACKPLANE, J5 CAN A, J6 CAN B, K1 FORCE-GUIDED 12V A, K2 FORCE-GUIDED 12V B, Q1 150V N-MOS, Q2 150V N-MOS, U1 LTC4368HMS-2, U2 ISOLATED 48V-12V 240W (TBD), U3 TPS26633RGE, U4 RPL-5.0 3V3/5A, U5 CH32V307VCT6, U6 ISO1042DW, U7 3V3-5V ISO 1W, U8 ESTOP DIAGNOSTIC OPTO, Y1 8MHz

Commit message: feat(hardware): implement EVT1 PCB power candidates
Parts:
- removed U2: ISOLATED 48V-12V 240W (TBD), WB:Isolated_48V_12V_240W_TBD, symbol controller:ISOLATED_DC_DC_TBD
- removed U7: 3V3-5V ISO 1W, Converter_DCDC:Converter_DCDC_muRata_MEJ1SxxxxSC_THT, symbol controller:MEJ1S0305SC
- added TP10: 3V3_PGOOD, TestPoint:TestPoint_Pad_D1.5mm, symbol controller:TESTPOINT
- added TP11: JETSON_PGOOD, TestPoint:TestPoint_Pad_D1.5mm, symbol controller:TESTPOINT
- added TP12: JETSON_FAULT_N, TestPoint:TestPoint_Pad_D1.5mm, symbol controller:TESTPOINT
- added TP13: U3_IMON, TestPoint:TestPoint_Pad_D1.5mm, symbol controller:TESTPOINT
- added TP14: ESTOP_A_MON, TestPoint:TestPoint_Pad_D1.5mm, symbol controller:TESTPOINT
- added TP15: ESTOP_B_MON, TestPoint:TestPoint_Pad_D1.5mm, symbol controller:TESTPOINT
- added TP9: 5V_CAN_ISO, TestPoint:TestPoint_Pad_D1.5mm, symbol controller:TESTPOINT
- added U2: 18-75V TO 12V 240W ISO, WB:Delta_Q36SR_QuarterBrick, symbol controller:DELTA_Q36SR
- added U7: 3V3-5V ISO 1W, WB:Murata_NXF1_MC, symbol controller:NXF1S0305MC
Connections:
- net 12V_ISO: now also U2.7 (+SENSE), U2.8 (+VOUT)
- net 3V3_LOGIC: now also U7.3 (+VIN)
- net 3V3_PGOOD: now also TP10.1 (TP)
- net 5V_CAN_ISO: now also TP9.1 (TP), U7.8 (+VOUT)
- net ESTOP_A_MON: now also TP14.1 (TP)
- net ESTOP_B_MON: now also TP15.1 (TP)
- net GND: now also U2.4 (-VOUT), U2.5 (-SENSE), U7.1 (-VIN)
- net GND_CAN_ISO: now also U7.7 (-VOUT)
- net GND_PWR: now also U2.2 (ON/OFF), U2.3 (-VIN)
- net JETSON_FAULT_N: now also TP12.1 (TP)
- net JETSON_PGOOD: now also TP11.1 (TP)
- net U3_IMON: now also TP13.1 (TP)
- net VBAT_PROTECTED: now also U2.1 (+VIN)
- no-connect marks 92 -> 89
